Commit message: adjusted inertia parameters to avoid uncontrollable spinning after collisions

File: sphero_description/robots/sphero.gazebo.xacro (robot description, xacro)
@@ -4,6 +4,6 @@
     <kp>100000000.0</kp>
     <kd>10.0</kd>
-    <mu1>0.1</mu1>
-    <mu2>0.1</mu2>
+    <mu1>0.04</mu1>
+    <mu2>0.04</mu2>
     <fdir1>1 0 0</fdir1>
     <maxVel>10.0</maxVel>
@@ -14,6 +14,6 @@
     <kp>100000000.0</kp>
     <kd>10.0</kd>
-    <mu1>10</mu1>
-    <mu2>10</mu2>
+    <mu1>0.04</mu1>
+    <mu2>0.04</mu2>
     <fdir1>1 0 0</fdir1>
     <maxVel>1.0</maxVel>
@@ -23,6 +23,6 @@
     <kp>100000000.0</kp>
     <kd>10.0</kd>
-    <mu1>10</mu1>
-    <mu2>10</mu2>
+    <mu1>0.04</mu1>
+    <mu2>0.04</mu2>
     <fdir1>1 0 0</fdir1>
     <maxVel>1.0</maxVel>
@@ -42,7 +42,7 @@
       <leftJoint>direction_joint</leftJoint>
       <rightJoint>rotation_joint</rightJoint>
-      <wheelSeparation>0.0381</wheelSeparation>
+      <wheelSeparation>0.025</wheelSeparation>
       <wheelDiameter>0.01</wheelDiameter>
-      <torque>20</torque>
+      <torque>0.025</torque>
       <commandTopic>/cmd_vel</commandTopic>
       <odometryTopic>/odom</odometryTopic>
@@ -69,9 +69,7 @@
   </gazebo>
   <!-- contact sensor -->
-  <!--
   <gazebo>
       <plugin name="gazebo_contact_sensor_plugin" filename="libgazebo_contact_sensor_plugin.so">
       </plugin>
   </gazebo>
-  -->
 </robot>

File: sphero_description/robots/sphero.urdf (robot description, URDF)
Before this commit: robot sphero, 3 links, 2 joints
Links:
- link base_direction_link: mass 0.05 -> 0.01
- link base_link: mass 0.5 -> 0.15; geometry collision sphere radius=0.03; visual sphere radius=0.01
- link base_rotation_link: mass 0.05 -> 0.01; geometry collision sphere radius=0.01; visual sphere radius=0.03
Joints:
- joint direction_joint: origin xyz=0.0 0.0 0.0 rpy=0 0 0 -> xyz=0 0 0 rpy=0 0 0
- joint rotation_joint: origin xyz=0.0 0.0 0.0 rpy=0 0 0 -> xyz=0 0 0 rpy=0 0 0

Commit message: fixed joint orientation in model definition

File: sphero_description/robots/sphero.gazebo.xacro (robot description, xacro)
@@ -42,6 +42,6 @@
       <leftJoint>direction_joint</leftJoint>
       <rightJoint>rotation_joint</rightJoint>
-      <wheelSeparation>0.025</wheelSeparation>
-      <wheelDiameter>0.02</wheelDiameter>
+      <wheelSeparation>0.0381</wheelSeparation>
+      <wheelDiameter>0.01</wheelDiameter>
       <torque>0.025</torque>
       <commandTopic>/cmd_vel</commandTopic>

File: sphero_description/robots/sphero.urdf (robot description, URDF)
Before this commit: robot sphero, 3 links, 2 joints
Joints:
- joint direction_joint: axis 1 0 0 -> -1 0 0

Commit message: adjusted movement to rotate around the correct axis

File: sphero_description/robots/sphero.gazebo.xacro (robot description, xacro)
@@ -4,6 +4,6 @@
     <kp>100000000.0</kp>
     <kd>10.0</kd>
-    <mu1>0.04</mu1>
-    <mu2>0.04</mu2>
+    <mu1>0.4</mu1>
+    <mu2>0.4</mu2>
     <fdir1>1 0 0</fdir1>
     <maxVel>10.0</maxVel>
@@ -23,6 +23,6 @@
     <kp>100000000.0</kp>
     <kd>10.0</kd>
-    <mu1>0.04</mu1>
-    <mu2>0.04</mu2>
+    <mu1>0.4</mu1>
+    <mu2>0.4</mu2>
     <fdir1>1 0 0</fdir1>
     <maxVel>1.0</maxVel>
@@ -43,10 +43,14 @@
       <rightJoint>rotation_joint</rightJoint>
       <wheelSeparation>0.0381</wheelSeparation>
-      <wheelDiameter>0.01</wheelDiameter>
+      <wheelDiameter>0.05</wheelDiameter>
+      <wheelAcceleration>0</wheelAcceleration>
+      <wheelTorque>0.02</wheelTorque>
       <torque>0.025</torque>
       <commandTopic>/cmd_vel</commandTopic>
       <odometryTopic>/odom</odometryTopic>
+      <positionTopic>Sphero1</positionTopic>
       <odometryFrame>/odom_frame</odometryFrame>
       <publishWheelJointState>true</publishWheelJointState>
+      <publishWheelTF>false</publishWheelTF>
       <odometrySource>world</odometrySource>
       <robotBaseFrame>base_link</robotBaseFrame>
@@ -65,5 +69,4 @@
       <updateRate>50.0</updateRate>
       <alwaysOn>true</alwaysOn>
-      <gaussianNoise>0</gaussianNoise>
     </plugin>
   </gazebo>

File: sphero_description/robots/sphero.urdf (robot description, URDF)
Before this commit: robot sphero, 3 links, 2 joints
Joints:
- joint direction_joint: axis -1 0 0 -> 0 1 0
- joint rotation_joint: limit lower=-1e+16 upper=1e+16 effort=18.85 velocity=0.2 -> lower=-1e+16 upper=1e+16 effort=18.85 velocity=1.57

Commit message: fixed simulation and adjusted for performance

File: sphero_description/robots/sphero.gazebo.xacro (robot description, xacro)
@@ -17,5 +17,5 @@
     <mu1>0.04</mu1>
     <mu2>0.04</mu2>
-    <fdir1>1 0 0</fdir1>
+    <fdir1>0 0 1</fdir1>
     <maxVel>1.0</maxVel>
     <minDepth>0.0005</minDepth>
@@ -68,5 +68,5 @@
       <gaussianNoise>0</gaussianNoise>
       <rpyOffsets>0 0 0</rpyOffsets>
-      <updateRate>50.0</updateRate>
+      <updateRate>50</updateRate>
       <alwaysOn>true</alwaysOn>
     </plugin>

File: sphero_description/robots/sphero.urdf (robot description, URDF)
Before this commit: robot sphero, 3 links, 2 joints
Joints:
- joint rotation_joint: limit lower=-1e+16 upper=1e+16 effort=18.85 velocity=1.57 -> effort=18.85 velocity=1.57; type revolute -> continuous
